Commit message: activate minus distance

File: collision_description/robots/panda.urdf.xacro (robot description, xacro)
@@ -3,8 +3,29 @@
   <xacro:arg name="arm_id" default="panda" />
   <xacro:arg name="hand" default="true" />
- <link name="world"/>
+  <link name="base">
+    <visual>
+      <origin xyz="-0.24 0 0.425" rpy="0 0 0"/>
+      <geometry>
+        <box size="0.6 0.9 0.85" />
+      </geometry>
+      <material name="White">
+        <color rgba="1.0 1.0 1.0 1.0"/>
+      </material>
+    </visual>
+    <collision>
+      <origin xyz="-0.24 0 0.425" rpy="0 0 0  "/>
+      <geometry>
+        <box size="0.6 0.9 0.85" />
+      </geometry>
+    </collision>
+  </link>
+  <xacro:include filename="env_box.xacro"/>
+  <xacro:box id="wall_1" connected_to="base" xyz="-0.59 0.3 1.0" size="0.1 0.33 2.0"/>
+  <xacro:box id="wall_2" connected_to="base" xyz="0.21 0.5 1.0" size="1.7 0.1 2.0"/>
+  <xacro:box id="table" connected_to="base" xyz="0.56 0.065 0.365" size="1.0 0.77 0.73"/>
+ <!-- <link name="world"/> -->
   <!-- single arm with gripper -->
   <xacro:include filename="$(find franka_description)/robots/common/franka_arm.xacro"/>
-  <xacro:franka_arm arm_id="$(arg arm_id)" connected_to="world"  xyz="0 0 0" gazebo="true"
+  <xacro:franka_arm arm_id="$(arg arm_id)" connected_to="base"  xyz="0 0 0.856" gazebo="true"
                     joint_limits="${xacro.load_yaml('$(find franka_description)/robots/panda/joint_limits.yaml')}"/>
   <xacro:if value="$(arg hand)">

File: collision_moveit_config/config/gazebo_panda.urdf (robot description, URDF)
Before this commit: robot panda, 23 links, 22 joints
Links:
- added link table, mass 0.1; collision box size=1.0 0.77 0.73; visual box size=1.0 0.77 0.73
- added link wall_1, mass 0.1; collision box size=0.1 0.33 2.0; visual box size=0.1 0.33 2.0
- added link wall_2, mass 0.1; collision box size=1.7 0.1 2.0; visual box size=1.7 0.1 2.0
- link base: geometry collision box size=0.6 0.9 0.85; visual box size=0.6 0.9 0.85
Joints:
- added joint base_table: type fixed, parent base, child table, origin xyz=0 0 0 rpy=0 0 0
- added joint base_wall_1: type fixed, parent base, child wall_1, origin xyz=0 0 0 rpy=0 0 0
- added joint base_wall_2: type fixed, parent base, child wall_2, origin xyz=0 0 0 rpy=0 0 0
- joint panda_joint_base: origin xyz=0 0 1.006 rpy=0 0 0 -> xyz=0 0 0.856 rpy=0 0 0

Commit message: add base

File: collision_description/robots/panda.urdf.xacro (robot description, xacro)
@@ -5,5 +5,6 @@
   <link name="base">
     <visual>
-      <origin xyz="-0.24 0 0.425" rpy="0 0 0"/>
+      <!-- <origin xyz="-0.24 0 0.425" rpy="0 0 0"/> -->
+      <origin xyz="0.085 0 0.425" rpy="0 0 0"/>
       <geometry>
         <box size="0.6 0.9 0.85" />
@@ -14,5 +15,6 @@
     </visual>
     <collision>
-      <origin xyz="-0.24 0 0.425" rpy="0 0 0  "/>
+      <!-- <origin xyz="-0.24 0 0.425" rpy="0 0 0  "/> -->
+      <origin xyz="0.085 0 0.425" rpy="0 0 0  "/>
       <geometry>
         <box size="0.6 0.9 0.85" />
@@ -20,8 +22,8 @@
     </collision>
   </link>
-  <xacro:include filename="env_box.xacro"/>
+  <!-- <xacro:include filename="env_box.xacro"/>
   <xacro:box id="wall_1" connected_to="base" xyz="-0.59 0.3 1.0" size="0.1 0.33 2.0"/>
   <xacro:box id="wall_2" connected_to="base" xyz="0.21 0.5 1.0" size="1.7 0.1 2.0"/>
-  <xacro:box id="table" connected_to="base" xyz="0.56 0.065 0.365" size="1.0 0.77 0.73"/>
+  <xacro:box id="table" connected_to="base" xyz="0.56 0.065 0.365" size="1.0 0.77 0.73"/> -->
  <!-- <link name="world"/> -->
   <!-- single arm with gripper -->
